Commit message: Add files via upload
Robot model

File: ten/urdf/ten.urdf (robot description, URDF)
Before this commit: robot ten, 11 links, 10 joints
Joints:
- joint joint_rl: limit lower=0 upper=0 effort=5 velocity=2 -> lower=-0.2 upper=0.2 effort=5 velocity=2
- joint joint_rr: limit lower=0 upper=0 effort=5 velocity=2 -> lower=-0.2 upper=0.2 effort=5 velocity=2
